File: hardware/kicad/osc_module/vinyl_adc_osc.kicad_pcb (KiCad board)
At the start: 2 copper layers, 40 x 44 mm, 8 parts, among them J1 DIP-8 PLUG, U9 74HCU04, Y1 6.144MHz

Commit message: finished digital addon board
Routing:
- net GND: track 116.5 -> 0.26 mm
- net Net-(R10-Pad2): track 59.5 -> 69.2 mm
- net Net-(C16-Pad1): track 52.7 -> 60.6 mm
- net Net-(C17-Pad1): track 25.4 -> 29.1 mm
- added copper zone on B.Cu, net GND
Other:
- board size 40 x 44 mm -> 41.9 x 44 mm

Commit message: Add solder mask ablation DXF and production files for osc module
Same flow as the digital board: 0.1 mm global mask expansion for
laser-to-board registration slack, mask_bottom.dxf generated from pad
geometry as closed circles/polylines for xTool fill-engraving (MASK =
openings, EDGE = outline for registration). Gerbers, drill, silk and
copper DXFs re-exported to match. Not mirrored - mirror in xTool with
the board copper-side up.
Other:
- rule pad_to_mask_clearance: 0 -> 0.1
Changed lines of the file:
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@@
 	)
 	(setup
-		(pad_to_mask_clearance 0)
+		(pad_to_mask_clearance 0.1)
 		(allow_soldermask_bridges_in_footprints no)
 		(tenting
