File: hardware/kicad/rev_d/vinyl_adc_rev_d.kicad_pcb (KiCad board)
At the start: 4 copper layers, 140 x 136 mm, 184 parts, among them J1 CLK SEL, J2 RASPBERRY PI 4, J20 LINE IN L, J22 TP L, J3 TONEARM GND, J4 GND LIFT, J5 TP DIG, J6 WP, J60 LINE IN R, J62 TP R, Q1 BC547, Q2 BC557, Q3 BC557, SW1 SHUTDOWN / WAKE GPIO3, SW2 USER GPIO23, U1 74HC244, U10 74HC244, U11 24LC32, U12 LM339, U2 LM358, U20 TL072, U21 LM311, U22 TL072, U23 74HC74, U24 74HC04, U3 74HCT132, U4 74HC4040, U6 74HC157, U60 TL072, U61 LM311, U62 TL072, U63 74HC74, U64 74HC04, U8 74HC4049, U9 74HCU04, Y1 6.144MHz

Commit message: Rev D ready for PCBWay: printable silkscreen, every legend back
The library footprints draw their outlines at 0.12 mm and the legends
used 0.135 mm strokes, both below PCBWay's 0.15 mm silkscreen minimum,
where lines can print broken or not at all. Every silkscreen stroke is
now at least 0.15 mm.

The new layout had also lost the labels that say what things are for:
LINE IN L/R, TONEARM GND, TRIM L/R, BOND on J4, the write jumper J6,
J1's 1-2 XTAL / 2-3 GPCLK, and the board title. They are placed next to
their parts, clear of every outline, and the six references with no free
spot are printed inside their outlines, under the body, where they can
be read during assembly.

DRC is still clean: no violations, no unconnected items, no warnings. The
production README now gives the copper layer order the 4-layer order form
asks for. Rev E's board is unchanged: the same legend pass leaves 16 of
its references off, so it needs its own silkscreen pass before ordering.
Other:
- board text added: "1-2 XTAL"
- board text added: "2-3 GPCLK"
- board text added: "BOND"
- board text added: "LINE IN L"
- board text added: "LINE IN R"
- board text added: "TONEARM GND"
- board text added: "TRIM L"
- board text added: "TRIM R"
- board text added: "VINYL ADC rev D through-hole Raspberry Pi 4 HAT"
- board text added: "WR: short"

Commit message: Rev D: sign it -- Mads Rudolph, madsrudolph.dev
"designed by Mads Rudolph / madsrudolph.dev 2026" on the component side
beside the board title, and the same line in the copper-side title block
under the Pi. DRC still clean: no violations, unconnected items or
warnings.
Other:
- board text added: "Mads Rudolph - madsrudolph.dev"
- board text added: "designed by Mads Rudolph"
- board text added: "madsrudolph.dev 2026"
Changed lines of the file:
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@@
 		(tags "C Disc series Radial pin pitch 5.00mm diameter 5mm width 2.5mm Capacitor")
 		(property "Reference" "C63"
-			(at 2.5 2.345 0)
+			(at -2.695 0 0)
 			(layer "F.SilkS")
 			(effects
@@
 		(tags "C Disc series Radial pin pitch 5.00mm diameter 5mm width 2.5mm Capacitor")
 		(property "Reference" "C64"
-			(at -2.695 0 0)
+			(at 6.895 0 90)
 			(layer "F.SilkS")
 			(effects
@@
 		)
 	)
+	(gr_text "madsrudolph.dev  2026"
+		(at 23.68 101.175 0)
+		(layer "F.SilkS")
+		(effects
+			(font
+				(size 1 1)
+				(thickness 0.15)
+			)
+		)
+	)
+	(gr_text "designed by Mads Rudolph"
+		(at 23.68 99.18 0)
+		(layer "F.SilkS")
+		(effects
+			(font
+				(size 1.1 1.1)
+				(thickness 0.165)
+			)
+		)
+	)
 	(gr_text "VINYL ADC  rev D  through-hole  Raspberry Pi 4 HAT"
 		(at 27.8 103.135 0)
@@
 		(layer "B.SilkS")
 		(effects
+			(font
+				(size 1 1)
+				(thickness 0.15)
+			)
+			(justify mirror)
+		)
+	)
+	(gr_text "Mads Rudolph  -  madsrudolph.dev"
+		(at 71.25 113.81 0)
+		(layer "B.SilkS")
+		(effects

Commit message: Rev D: final silkscreen text adjustments, exported for PCBWay
Hand edits to the legend positions in KiCad (the signature moved to the
centre of the lower strip). DRC with zones refilled: no violations, no
unconnected items.
Parts:
- moved J2 55.4 mm to (139.8, 78.1)
- moved C1 55.4 mm to (145.3, 84.5)
- moved C10 55.4 mm to (165.3, 63.2)
- moved C11 55.4 mm to (174.6, 59.8)
- moved C13 55.4 mm to (143.6, 59.8)
- moved C15 55.4 mm to (143.6, 50.8)
- moved C16 55.4 mm to (162.1, 33.2)
- moved C17 55.4 mm to (164.3, 39.5)
- moved C18 55.4 mm to (146.1, 124.8)
- moved C19 55.4 mm to (138.3, 124.8)
- moved C2 55.4 mm to (140.1, 87.2)
- moved C20 55.4 mm to (61.8, 53.8)
- moved C21 55.4 mm to (54.3, 59.0)
- moved C22 55.4 mm to (100.8, 38.2)
- moved C23 55.4 mm to (74.6, 59.8)
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