File: hardware/kicad/rev_c/vinyl_adc_rev_c.kicad_sch (KiCad schematic)
At the start: 111 parts, among them J1 CLK SEL, J2 RASPBERRY PI 4, J20 LINE IN L, J60 LINE IN R, U1 74HC244, U2 LM358, U20 TL072, U21 LM311, U22 TL072, U23 74HC74, U24 74HC04, U3 74HCT132, U4 74HC4040, U6 74HC157, U60 TL072, U61 LM311, U62 TL072, U63 74HC74, U64 74HC04, U8 74HC4049, U9 74HCU04, Y1 6.144MHz

Commit message: Rev D enclosure, short v2 and channel L Gerbers
Rev D enclosure: CAD scripts, spec, print files (STL/3MF/STEP/DXF) and the
SolidCraft assembly with renders. Short v2: the Remotion project, voice/sfx
scripts and PCB layer art (renders, audio and footage stay local). Channel L
production Gerbers, bring-up log update and KiCad project tweaks.
Other:
- moved on the sheet: C1, C10, C11, C13, C15, C16, C17, C2, C20, C21, C22, C23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
